Commit message: Added control plugin, gz_bridge, and teleoperation

File: description/robot_core.xacro (robot description, xacro)
@@ -47,4 +47,5 @@
     <origin xyz="0 0.175 0" rpy="-${pi/2} 0 0"/>
     <axis xyz="0 0 1"/>
+    <limit effort="0.05" velocity="10.0"/>
   </joint>
   <link name="left_wheel">
@@ -70,4 +71,5 @@
     <origin xyz="0 -0.175 0" rpy="${pi/2} 0 0"/>
     <axis xyz="0 0 -1"/>
+    <limit effort="0.05" velocity="10.0"/>
   </joint>
   <link name="right_wheel">
@@ -109,3 +111,7 @@
     </xacro:inertial_sphere>
   </link>
+  <gazebo reference="caster_wheel">
+    <mu1 value="0.0"/>
+    <mu2 value="0.0"/>
+  </gazebo>
 </robot>
